Commit message: Update diffdrive URDF and add gazebo racetrack world

File: src/echo_description/diffdrive_urdf/robot_core.xacro (robot description, xacro)
@@ -30,4 +30,12 @@
                <box size="${lx} ${ly} ${lz}"/>
             </geometry>
+             <surface>
+                <friction>
+                <ode>
+                    <mu>1.0</mu>
+                    <mu2>1.0</mu2>
+                </ode>
+                </friction>
+            </surface>
         </collision>
         <xacro:inertial_box mass="5.0" x="${lx}" y="${ly}" z="${lz}">
@@ -53,6 +61,14 @@
         <collision>
             <geometry>
-                  <sphere radius="${rad_w}" />
+                  <cylinder radius="${rad_w}" length="${le_w}"/>
             </geometry>
+             <surface>
+                <friction>
+                <ode>
+                    <mu>1.0</mu>
+                    <mu2>1.0</mu2>
+                </ode>
+                </friction>
+            </surface>
         </collision>
         <xacro:inertial_cylinder mass="0.1" length="${le_w}" radius="${rad_w}">
@@ -78,5 +94,5 @@
         <collision>
             <geometry>
-                  <sphere radius="${rad_w}" />
+                  <cylinder radius="${rad_w}" length="${le_w}"/>
             </geometry>
         </collision>

Commit message: Added line segment Exctraction

File: src/echo_description/diffdrive_urdf/robot_core.xacro (robot description, xacro)
@@ -8,4 +8,6 @@
     <xacro:property name="lx" value="0.4"/>
     <xacro:property name="lz" value="0.05"/>
+    <xacro:property name="chassis_mass" value="5.8"/>
+    <xacro:property name="wheel_mass" value="0.5"/>
     <!-- Example link -->
     <link name="base_link">
@@ -31,5 +33,5 @@
             </geometry>
         </collision>
-        <xacro:inertial_box mass="5.0" x="${lx}" y="${ly}" z="${lz}">
+        <xacro:inertial_box mass="${chassis_mass}" x="${lx}" y="${ly}" z="${lz}">
             <origin xyz="0 0 0" rpy="0 0 0"/>
         </xacro:inertial_box>
@@ -56,5 +58,5 @@
             </geometry>
         </collision>
-        <xacro:inertial_cylinder mass="0.1" length="${le_w}" radius="${rad_w}">
+        <xacro:inertial_cylinder mass="${wheel_mass}" length="${le_w}" radius="${rad_w}">
             <origin xyz="0 0 0" rpy="0 0 0"/>
         </xacro:inertial_cylinder>
@@ -81,5 +83,5 @@
             </geometry>
         </collision>
-        <xacro:inertial_cylinder mass="0.1" length="${le_w}" radius="${rad_w}">
+        <xacro:inertial_cylinder mass="${wheel_mass}" length="${le_w}" radius="${rad_w}">
             <origin xyz="0 0 0" rpy="0 0 0"/>
         </xacro:inertial_cylinder>
@@ -147,3 +149,19 @@
         </xacro:inertial_sphere>
     </link>
+    <gazebo reference="left_wheel">
+        <mu1>2.0</mu1>
+        <mu2>2.0</mu2>
+    </gazebo>
+    <gazebo reference="right_wheel">
+        <mu1>2.0</mu1>
+        <mu2>2.0</mu2>
+    </gazebo>
+    <gazebo reference="caster_rear_wheel">
+        <mu1>2.0</mu1>
+        <mu2>2.0</mu2>
+    </gazebo>
+    <gazebo reference="caster_front_wheel">
+        <mu1>2.0</mu1>
+        <mu2>2.0</mu2>
+    </gazebo>
 </robot>
